File: Controller-Tennis/PCB/controller-tennis/controller-tennis.kicad_pcb (KiCad board)
At the start: 2 copper layers, 84 x 37 mm, 7 parts, among them SW1 SW_Push, U1 ESP32-C3_SUPERMINI_TH

Commit message: status quo
not working, all kap00t
Parts:
- added G***: LOGO, LOGO, B.Cu at (181.6, 114.0)
- added G***: LOGO, LOGO, B.Cu at (138.4, 112.7)
Routing:
- net GND: vias 0 -> 18
Other:
- outline, holes or cut-outs redrawn
