File: Machine/PCB/arcade-pcb/arcade-pcb.kicad_pcb (KiCad board)
At the start: 2 copper layers, 33 x 35 mm, 4 parts, among them SW1 SW_Push, U1 ESP32-C3_SUPERMINI_TH

Commit message: status quo
not working, all kap00t
Parts:
- added BZ1: Buzzer, Buzzer_Beeper:Buzzer_12x9.5RM7.6, B.Cu at (143.1, 76.6)
- added R1: 100R, Resistor_THT:R_Axial_DIN0207_L6.3mm_D2.5mm_P7.62mm_Horizontal, F.Cu at (133.6, 75.7)
- Display1: footprint Connector_PinHeader_2.54mm:PinHeader_1x07_P2.54mm_Vertical -> ehajo-footprints:PinHeader_1x07_P1.27mm_Vertical_hand
- moved Display1 3.84 mm to (143.2, 84.9)
- moved U1 0.22 mm to (147.0, 71.7)
Connections:
- U1 pad 20: unconnected-(U1-GPIO20-Pad20) -> Net-(U1-GPIO20)
Routing:
- net Net-(BZ1-+): track 0.00 -> 14.4 mm
- net Net-(U1-GPIO20): track 0.00 -> 6.35 mm
- net +3.3V: track 27.3 -> 24.6 mm
- net /CS: track 31.6 -> 29.9 mm
- net /DC: track 18.8 -> 19.9 mm
- net /RES: track 9.28 -> 9.94 mm
- net /DOUT: track 5.16 -> 5.81 mm
- net /MISO: track 31.3 -> 30.7 mm
- net GND: vias 22 -> 18
Other:
- outline, holes or cut-outs redrawn
- board text added: "Arcade-Machine v1.1"
- board text removed: "Arcade-Machine v1.0"

Commit message: aktueller stand
Parts:
- added G***: LOGO, LOGO, B.Cu at (136.4, 89.4)
- Display1, R1, SW1, WS2812: moved to B.Cu
- moved SW1 4.62 mm to (144.7, 91.2), turned to 0 degrees
- moved BZ1 3.88 mm to (147.0, 76.6)
- turned Display1 to -90 degrees
- turned WS2812 to 180 degrees
Routing:
- net Net-(U1-GPIO10): track 34.8 -> 28.5 mm
Other:
- board text added: "Arcade-Machine v1.2"
- board text added: "Get Ready Player 1"
- board text removed: "Arcade-Machine v1.1"
